Commit message: Remove old Dual_arm_art artifacts and recordings, both robot picking successfully

File: configs/urdfs/panda_drake2.urdf (robot description, URDF)
Before this commit: robot panda, 12 links, 11 joints
Joints:
- joint robot_to_world: origin xyz=-0.5 0.0 0.0 rpy=0.0 0.0 3.14 -> xyz=0.5 0.0 0.0 rpy=0.0 0.0 3.14159
